File: KiCad/AISReceiver.kicad_pcb (KiCad board)
At the start: 2 copper layers, 26.7 x 24.8 mm, 14 parts, among them P1 Antenna, P2 Power, P3 SPI, P4 GPIO, U1 SI4362, X1 30 MHz

Commit message: Rev B schematic and layout
Parts:
- added C4: 220 pF, SM0805, F.Cu at (113.5, 88.6)
- added R2: 100 K, SM0805, F.Cu at (129.0, 94.0)
- CR1: value 11.5-13.8 pF -> 10 pF
- CR2: value 6-7 pF -> 5 pF
- LR1: value 270 nH -> 280 nH
- LR2: value 160 nH -> 200 nH
- X1: footprint crystal_FA238-TSX3225 -> Crystal-50x32
- moved P1 134.8 mm to (113.5, 83.3)
- moved C3 133.5 mm to (115.8, 95.2), turned to 270 degrees
- moved CR2 133.3 mm to (117.1, 89.7)
- moved P3 133.1 mm to (133.9, 93.5)
- moved X1 133.1 mm to (127.8, 83.3)
- moved P2 133.1 mm to (114.8, 99.8)
- moved P4 133.1 mm to (125.0, 99.8)
- moved U1 133.1 mm to (125.0, 89.7)
- moved C1 132.6 mm to (121.4, 95.2)
- moved C2 132.4 mm to (118.6, 95.2), turned to 270 degrees
- moved CR1 131.7 mm to (118.1, 83.6), turned to 270 degrees
- moved LR2 131.4 mm to (117.1, 86.9), turned to 180 degrees
- moved LR1 130.3 mm to (120.4, 88.9)
- moved R1 119.0 mm to (129.0, 96.5), turned to 0 degrees
Connections:
- CR2 pad 1: N-0000019 -> N-0000021
- LR2 pad 2: N-0000019 -> N-0000021
- P1 pad 1: N-0000019 -> N-0000016
- P4 pad 1: N-000007 (its old number) -> N-0000010
- P4 pad 2: N-000006 -> N-0000013
- U1 pad 10: N-000007 (its old number) -> N-0000013
- U1 pad 9: N-000006 -> N-0000010
Routing:
- net GND: track 16.2 -> 50.7 mm, vias 8 -> 24
- net /GPIO3: track 41.4 -> 23.1 mm
- net /GPIO2: track 36.9 -> 18.8 mm
- net /SDN: track 42.0 -> 27.2 mm
- net N-0000010: track 0.00 -> 10.1 mm, vias 0 -> 1
- net N-000007 (its old number): track 9.32 -> 0.00 mm
- net N-000006: track 8.48 -> 0.00 mm
- net N-0000013: track 0.00 -> 8.27 mm
- net N-0000019: track 7.27 -> 0.00 mm
- net N-000002: track 13.4 -> 7.95 mm
- net N-0000021: track 0.00 -> 5.42 mm
- net N-0000014: track 8.39 -> 13.0 mm, vias 0 -> 1
- net N-0000016: track 0.00 -> 3.11 mm
- net N-0000017: track 7.76 -> 4.78 mm
- net N-000008: track 4.04 -> 3.20 mm
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- added copper zone on F.Cu, net GND
Other:
- board size 26.7 x 24.8 mm -> 25.4 x 22.9 mm
- board text added: "ANT"
