File: KiCad/AISReceiver.sch (KiCad schematic (older format))
At the start: 15 parts, among them P1 Antenna, P2 Power, P3 SPI, P4 GPIO, U1 SI4362, X1 30 MHz

Commit message: Rev B schematic and layout
Parts:
- added C4: 220 pF, ~, symbol C
- CR1: value 10 pF -> 12 pF
- CR2: value 5 pF -> 6 pF
- LR1: value 280 nH -> 240 nH
Connections:
- wire segments 51 -> 52
Changed lines of the file:
@@
 encoding utf-8
 Sheet 1 1
-Title ""
-Date "28 dec 2013"
-Rev ""
+Title "Si4362 Breakout"
+Date "19 jan 2014"
+Rev "B"
 Comp ""
 Comment1 ""
@@
 P 3700 2200
 F 0 "CR1" H 3700 2300 40  0000 L CNN
-F 1 "10 pF" H 3706 2115 40  0000 L CNN
+F 1 "12 pF" H 3706 2115 40  0000 L CNN
 F 2 "~" H 3738 2050 30  0000 C CNN
 F 3 "~" H 3700 2200 60  0000 C CNN
@@
 P 3300 3400
 F 0 "CR2" H 3300 3500 40  0000 L CNN
-F 1 "5 pF" H 3306 3315 40  0000 L CNN
+F 1 "6 pF" H 3306 3315 40  0000 L CNN
 F 2 "~" H 3338 3250 30  0000 C CNN
 F 3 "~" H 3300 3400 60  0000 C CNN
@@
 P 3700 3000
 F 0 "LR1" V 3650 3000 40  0000 C CNN
-F 1 "280 nH" V 3800 3000 40  0000 C CNN
+F 1 "240 nH" V 3800 3000 40  0000 C CNN
 F 2 "~" H 3700 3000 60  0000 C CNN
 F 3 "~" H 3700 3000 60  0000 C CNN
@@
 	5500 4250 5300 4250
 Connection ~ 5300 4250
-Wire Wire Line
-	1950 3400 3100 3400
 $Comp
 L R R2
@@
 Connection ~ 6850 3400
 $Comp
-L GND #PWR?
+L GND #PWR06
 U 1 1 527EDCFC
 P 6850 1800
-F 0 "#PWR?" H 6850 1800 30  0001 C CNN
+F 0 "#PWR06" H 6850 1800 30  0001 C CNN
 F 1 "GND" H 6850 1730 30  0001 C CNN
 F 2 "" H 6850 1800 60  0000 C CNN
@@
 Wire Wire Line
 	6400 4200 7100 4200
+$Comp
+L C C4
+U 1 1 52D481B6
+P 2400 3400
+F 0 "C4" H 2400 3500 40  0000 L CNN
+F 1 "220 pF" H 2406 3315 40  0000 L CNN
+F 2 "~" H 2438 3250 30  0000 C CNN
+F 3 "~" H 2400 3400 60  0000 C CNN
+	1    2400 3400
+	0    -1   -1   0
+$EndComp
+Wire Wire Line
+	2600 3400 3100 3400
+Wire Wire Line
+	2200 3400 1950 3400
 $EndSCHEMATC
